Commit message: change robot model

File: src/gazebo_r2d2/urdf/r2d2.urdf.xacro (robot description, xacro)
@@ -1,63 +1,89 @@
 <?xml version="1.0"?>
 <robot name="r2d2" xmlns:xacro="http://ros.org/wiki/xacro">
-  <!-- macro template -->
-  <xacro:include filename="$(find gazebo_r2d2)/urdf/utils.urdf.xacro" />
-  <!-- link -->
-  <xacro:link_cylinder_no_ineatia link_name="axis" radius="0.01" length="0.5">
-    <origin xyz="0 0 0" rpy="1.57 0 0" />
-  </xacro:link_cylinder_no_ineatia>
-  <xacro:link_box link_name="leg1" width="0.20" height="0.10" depth="0.8">
-    <origin xyz="0 0 -0.3" />
-  </xacro:link_box>
-  <xacro:link_box link_name="leg2" width="0.20" height="0.10" depth="0.8">
-    <origin xyz="0 0 -0.3" />
-  </xacro:link_box>
-  <xacro:link_cylinder link_name="body" radius="0.20" length="0.6">
-      <origin xyz="0 0 -0.2" />
-  </xacro:link_cylinder>
-  <xacro:link_sphere link_name="head" radius="0.40">
-      <origin/>
-  </xacro:link_sphere>
-  <xacro:link_cylinder link_name="rod" radius="0.02" length="0.2">
-      <origin xyz="0 0 -0.1" />
-  </xacro:link_cylinder>
-  <xacro:link_box link_name="box" width="0.05" height="0.05" depth="0.05">
-      <origin/>
-  </xacro:link_box>
-  <!-- joint -->
-  <joint name="leg1connect" type="fixed">
-    <origin xyz="0 .30 0" />
-    <parent link="axis"/>
-    <child link="leg1"/>
+  <xacro:property name="width" value="0.2" />
+  <xacro:property name="leglen" value="0.6" />
+  <xacro:property name="polelen" value="0.2" />
+  <xacro:property name="bodylen" value="0.6" />
+  <xacro:property name="baselen" value="0.4" />
+  <xacro:property name="wheeldiam" value="0.07" />
+  <xacro:include filename="$(find gazebo_r2d2)/urdf/utils.urdf.xacro"/>
+  <link name="base_link">
+    <visual>
+      <geometry>
+        <cylinder radius="${width}" length="${bodylen}"/>
+      </geometry>
+      <material name="blue"/>
+    </visual>
+    <collision>
+      <geometry>
+        <cylinder radius="${width}" length="${bodylen}"/>
+      </geometry>
+    </collision>
+    <xacro:default_inertial mass="10"/>
+  </link>
+  <xacro:leg prefix="right" reflect="-1" />
+  <xacro:leg prefix="left" reflect="1" />
+  <link name="head">
+    <visual>
+      <geometry>
+        <sphere radius="${width}"/>
+      </geometry>
+      <material name="white"/>
+    </visual>
+    <collision>
+      <geometry>
+        <sphere radius="${width}"/>
+      </geometry>
+    </collision>
+    <xacro:default_inertial mass="2"/>
+  </link>
+  <joint name="head_swivel" type="fixed">
+    <parent link="base_link"/>
+    <child link="head"/>
+    <origin xyz="0 0 ${bodylen/2}"/>
   </joint>
-  <joint name="leg2connect" type="fixed">
-    <origin xyz="0 -.30 0" />
-    <parent link="axis"/>
-    <child link="leg2"/>
+  <link name="box">
+    <visual>
+      <geometry>
+        <box size="0.08 0.08 0.08"/>
+      </geometry>
+      <material name="blue"/>
+      <origin xyz="-0.04 0 0"/>
+    </visual>
+    <collision>
+      <geometry>
+        <box size="0.08 0.08 0.08"/>
+      </geometry>
+    </collision>
+    <xacro:default_inertial mass="1"/>
+  </link>
+  <joint name="tobox" type="fixed">
+    <parent link="head"/>
+    <child link="box"/>
+    <origin xyz="${.707*width+0.04} 0 ${.707*width}"/>
   </joint>
-  <joint name="tilt" type="revolute">
-    <parent link="axis"/>
-    <child link="body"/>
-    <origin xyz="0 0 0" rpy="0 0 0" />
-    <axis xyz="0 1 0" />
-    <limit upper="0" lower="-.5" effort="10" velocity="10" />
-  </joint>
-  <joint name="swivel" type="continuous">
-    <origin xyz="0 0 0.1" />
-    <axis xyz="0 0 1" />
-    <parent link="body"/>
-    <child link="head"/>
-  </joint>
-  <joint name="periscope" type="prismatic">
-    <origin xyz=".12 0 .15" />
-    <axis xyz="0 0 1" />
-    <limit upper="0" lower="-.5" effort="10" velocity="10" />
-    <parent link="head"/>
-    <child link="rod"/>
-  </joint>
-  <joint name="boxconnect" type="fixed">
-    <origin xyz="0 0 0" />
-    <parent link="rod"/>
-    <child link="box"/>
-  </joint>
+  <!-- Gazebo plugin for ROS Control -->
+  <gazebo>
+    <plugin name="gazebo_ros_control" filename="libgazebo_ros_control.so">
+      <robotNamespace>/</robotNamespace>
+    </plugin>
+    <plugin name='front_diff_drive' filename='libgazebo_ros_diff_drive.so'>
+      <update_rate>50</update_rate>
+      <left_joint>left_front_wheel_joint</left_joint>
+      <right_joint>right_front_wheel_joint</right_joint>
+      <wheel_separation>${width}</wheel_separation>
+      <wheel_diameter>${wheeldiam/2}</wheel_diameter>
+      <robot_base_frame>base_link</robot_base_frame>
+			<publishWheelJointState>true</publishWheelJointState>
+    </plugin>
+    <plugin name='back_diff_drive' filename='libgazebo_ros_diff_drive.so'>
+      <update_rate>50</update_rate>
+      <left_joint>left_back_wheel_joint</left_joint>
+      <right_joint>right_back_wheel_joint</right_joint>
+      <wheel_separation>${width}</wheel_separation>
+      <wheel_diameter>${wheeldiam/2}</wheel_diameter>
+      <robot_base_frame>base_link</robot_base_frame>
+			<publishWheelJointState>true</publishWheelJointState>
+    </plugin>
+  </gazebo>
 </robot>

File: src/gazebo_r2d2/urdf/utils.urdf.xacro (robot description, xacro)
@@ -1,90 +1,106 @@
 <?xml version="1.0"?>
 <robot name="r2d2" xmlns:xacro="http://ros.org/wiki/xacro">
-  <xacro:macro name="material_white">
-    <material name="white">
-      <color rgba="1 1 1 1"/>
-    </material>
-  </xacro:macro>
-  <xacro:macro name="simple_inertia">
+  <material name="blue">
+    <color rgba="0 0 0.8 1"/>
+  </material>
+  <material name="black">
+    <color rgba="0 0 0 1"/>
+  </material>
+  <material name="white">
+    <color rgba="1 1 1 1"/>
+  </material>
+  <xacro:macro name="default_inertial" params="mass">
     <inertial>
-      <mass value="1"/>
-      <inertia ixx="100" ixy="0" ixz="0" iyy="100" iyz="0" izz="100" />
-      <origin/>
+      <mass value="${mass}" />
+      <inertia ixx="1.0" ixy="0.0" ixz="0.0" iyy="1.0" iyz="0.0" izz="1.0" />
     </inertial>
   </xacro:macro>
-  <xacro:macro name="link_cylinder_no_ineatia" params="link_name radius length *origin">
-    <link name="${link_name}">
+  <xacro:macro name="wheel" params="prefix suffix reflect">
+    <link name="${prefix}_${suffix}_wheel">
       <visual>
-        <xacro:insert_block name="origin"/>
+        <origin xyz="0 0 0" rpy="${pi/2} 0 0" />
         <geometry>
-          <cylinder radius="${radius}" length="${length}" />
+          <cylinder radius="${wheeldiam/2}" length="0.1"/>
         </geometry>
-        <xacro:material_white />
+        <material name="black"/>
       </visual>
       <collision>
-        <xacro:insert_block name="origin"/>
+        <origin xyz="0 0 0" rpy="${pi/2} 0 0" />
         <geometry>
-          <cylinder radius="${radius}" length="${length}" />
+          <cylinder radius="${wheeldiam/2}" length="0.1"/>
         </geometry>
-        <contact_coefficients mu="0" kp="1000.0" kd="1.0"/>
       </collision>
+      <xacro:default_inertial mass="1"/>
     </link>
+    <joint name="${prefix}_${suffix}_wheel_joint" type="continuous">
+      <axis xyz="0 1 0" rpy="0 0 0" />
+      <parent link="${prefix}_base"/>
+      <child link="${prefix}_${suffix}_wheel"/>
+      <origin xyz="${baselen*reflect/3} 0 -${wheeldiam/2+.05}" rpy="0 0 0"/>
+    </joint>
+    <!-- This block provides the simulator (Gazebo) with information on a few additional
+    physical properties. See http://gazebosim.org/tutorials/?tut=ros_urdf for more-->
+    <gazebo reference="${prefix}_${suffix}_wheel">
+      <mu1 value="1.0"/>
+      <mu2 value="1.0"/>
+      <kp value="10000000.0" />
+      <kd value="1.0" />
+      <material>Gazebo/Grey</material>
+    </gazebo>
+    <!-- This block connects the wheel joint to an actuator (motor), which informs both
+    simulation and visualization of the robot -->
+    <transmission name="${prefix}_${suffix}_wheel_trans">
+      <type>transmission_interface/SimpleTransmission</type>
+      <actuator name="${prefix}_${suffix}_wheel_motor">
+        <mechanicalReduction>1</mechanicalReduction>
+      </actuator>
+      <joint name="${prefix}_${suffix}_wheel_joint">
+        <hardwareInterface>hardware_interface/VelocityJointInterface</hardwareInterface>
+      </joint>
+    </transmission>
   </xacro:macro>
-  <xacro:macro name="link_cylinder" params="link_name radius length *origin">
-    <link name="${link_name}">
-      <xacro:simple_inertia/>
+  <xacro:macro name="leg" params="prefix reflect">
+    <link name="${prefix}_leg">
       <visual>
-        <xacro:insert_block name="origin"/>
         <geometry>
-          <cylinder radius="${radius}" length="${length}" />
+          <box size="${leglen} 0.1 0.2"/>
         </geometry>
-        <xacro:material_white />
+        <origin xyz="0 0 -${leglen/2}" rpy="0 ${pi/2} 0"/>
+        <material name="white"/>
       </visual>
       <collision>
-        <xacro:insert_block name="origin"/>
         <geometry>
-          <cylinder radius="${radius}" length="${length}" />
+          <box size="${leglen} 0.1 0.2"/>
         </geometry>
-        <contact_coefficients mu="0" kp="1000.0" kd="1.0"/>
+        <origin xyz="0 0 -${leglen/2}" rpy="0 ${pi/2} 0"/>
       </collision>
+      <xacro:default_inertial mass="10"/>
     </link>
-  </xacro:macro>
-  <xacro:macro name="link_box" params="link_name width height depth *origin">
-    <link name="${link_name}">
-      <xacro:simple_inertia/>
+    <joint name="base_to_${prefix}_leg" type="fixed">
+      <parent link="base_link"/>
+      <child link="${prefix}_leg"/>
+      <origin xyz="0 ${reflect*(width+.02)} 0.25" />
+    </joint>
+    <link name="${prefix}_base">
       <visual>
-        <xacro:insert_block name="origin"/>
         <geometry>
-          <box size="${width} ${height} ${depth}" />
+          <box size="${baselen} 0.1 0.1"/>
         </geometry>
-        <xacro:material_white />
+        <material name="white"/>
       </visual>
       <collision>
-        <xacro:insert_block name="origin"/>
         <geometry>
-          <box size="${width} ${height} ${depth}" />
+          <box size="${baselen} 0.1 0.1"/>
         </geometry>
-        <contact_coefficients mu="0" kp="1000.0" kd="1.0"/>
       </collision>
+      <xacro:default_inertial mass="10"/>
     </link>
-  </xacro:macro>
-  <xacro:macro name="link_sphere" params="link_name radius *origin">
-    <link name="${link_name}">
-      <xacro:simple_inertia/>
-      <visual>
-        <xacro:insert_block name="origin"/>
-        <geometry>
-          <sphere radius=".4" />
-        </geometry>
-        <material name="white" />
-      </visual>
-      <collision>
-        <xacro:insert_block name="origin"/>
-        <geometry>
-          <sphere radius=".4" />
-        </geometry>
-        <contact_coefficients mu="0" kp="1000.0" kd="1.0"/>
-      </collision>
-    </link>
+    <joint name="${prefix}_base_joint" type="fixed">
+      <parent link="${prefix}_leg"/>
+      <child link="${prefix}_base"/>
+      <origin xyz="0 0 ${-leglen}" />
+    </joint>
+    <xacro:wheel prefix="${prefix}" suffix="front" reflect="1"/>
+    <xacro:wheel prefix="${prefix}" suffix="back" reflect="-1"/>
   </xacro:macro>
 </robot>
