Commit message: mod diffbot

File: src/r2d2_control/urdf/r2d2_ros2_control_with_diffbotsystem.urdf.xacro (robot description, xacro)
@@ -26,33 +26,4 @@
   <xacro:ros2_control_system suffix="front" />
   <xacro:ros2_control_system suffix="back" />
-  <ros2_control name="front_wheel_system" type="system">
-    <!-- Need clone and build https://github.com/ros-controls/ros2_control_demos -->
-    <hardware>
-      <plugin>ros2_control_demo_hardware/DiffBotSystemHardware</plugin>
-      <param name="example_param_hw_start_duration_sec">2.0</param>
-      <param name="example_param_hw_stop_duration_sec">3.0</param>
-    </hardware>
-    <!-- for diff_drive_controller -->
-    <!-- https://github.com/ros-controls/ros2_controllers/blob/master/diff_drive_controller/src/diff_drive_controller.cpp#L122-L144 -->
-    <!-- Need velocity command interface and position state interface-->
-    <joint name="left_front_wheel_joint">
-      <command_interface name="velocity">
-        <param name="min">-1</param>
-        <param name="max"> 1</param>
-      </command_interface>
-      <!-- DiffBotSystemHardware need two states -->
-      <state_interface name="position"/>
-      <state_interface name="velocity"/>
-    </joint>
-    <joint name="right_front_wheel_joint">
-      <command_interface name="velocity">
-        <param name="min">-1</param>
-        <param name="max"> 1</param>
-      </command_interface>
-      <!-- DiffBotSystemHardware need two states -->
-      <state_interface name="position"/>
-      <state_interface name="velocity"/>
-    </joint>
-  </ros2_control>
   <link name="head">
     <visual>
